File: Hardware/Board.brd (EAGLE design)
At the start: 169.8 x 111.2 mm, 103 parts, among them IC1 BD5229G-TR, IC4 XC6220A331MR-G, J1 FH34SRJ-24S-0.5SH_99_, J2 SAMACSYS_PARTS_USB4110-GF-A, J3 QWIIC_RIGHT_ANGLE, J4 112A-TAAR-R03_ATTEND, Q1 20V/4.2A/52mΩ/1.4W, Q2 20V/4.2A/52mΩ/1.4W, Q3 SI1308EDL-T1-GE3, U1 ESP32_WROVER_SPARKFUN-IC-POWE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

Commit message: finished board
Parts:
- moved L1 1.35 mm to (81.3, 31.7)
- moved RESET_BUTTON 0.82 mm to (24.2, 107.8)
- moved BOOT_BUTTON 0.74 mm to (49.2, 107.8)
Routing:
- net 3V3: track 471.9 -> 553.6 mm, vias 13 -> 8
- net IO/CHANGE: track 75.0 -> 124.5 mm, vias 2 -> 0
- net EPD_3V3: track 117.3 -> 80.1 mm, vias 3 -> 4
- net SCK: track 230.8 -> 196.8 mm, vias 8 -> 7
- net N$12: track 39.8 -> 8.29 mm
- net VUSB: track 0.00 -> 30.4 mm, vias 0 -> 3
- net RESET: track 102.7 -> 130.8 mm, vias 2 -> 0
- net N$10: track 56.1 -> 31.4 mm
- net GND: track 749.0 -> 724.6 mm, vias 15 -> 5
- net EPD_RST: track 126.5 -> 106.6 mm, vias 4 -> 2
- net EPD_DC: track 133.0 -> 114.4 mm, vias 0 -> 2
- net RTC_RST: track 68.8 -> 86.4 mm
- net EPD_3V3_C: track 121.4 -> 103.9 mm
- net I2C_PW: track 167.3 -> 184.7 mm
- net PREVGH: track 38.2 -> 22.5 mm, vias 5 -> 2
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- added copper zone on layer 1, net GND
- added copper zone on layer 16, net GND
